File: A-10CV1.1/A-10C-UFC/A-10C-UFC.kicad_pcb (KiCad board)
At the start: 2 copper layers, 257.7 x 65.9 mm, 42 parts, among them J1 Conn_01x08_MountingPin, J2 Conn_01x10_MountingPin, J3 Conn_01x06_MountingPin, J4 Conn_01x15_Female, J5 Conn_01x15_Female, SW1 SW_Push, SW10 SW_Push, SW11 SW_Push, SW12 SW_Push, SW13 SW_Push, SW14 SW_Push, SW15 SW_Push, SW16 SW_Push, SW17 SW_Push, SW18 SW_Push, SW19 SW_Push, SW2 SW_Push, SW20 SW_Push, SW21 SW_Push, SW22 SW_Push, SW23 SW_Push, SW24 SW_Push, SW25 SW_Push, SW26 SW_Push, SW27 SW_Push, SW28 SW_Push, SW29 SW_Push, SW3 SW_Push, SW30 SW_Push, SW31 SW_Push, SW32 SW_Push, SW33 SW_Push, SW34 SW_Push, SW35 SW_Push, SW4 SW_Push, SW5 SW_Push, SW6 SW_Push, SW7 SW_Push, SW8 SW_Push, SW9 SW_Push

Commit message: Updated for multi aircraft capability.  Added wiring and code.
Parts:
- added J6: Conn_01x08_MountingPin, Connector_PinHeader_2.54mm:PinHeader_1x08_P2.54mm_Vertical, B.Cu at (279.4, 66.3)
- added J7: Conn_01x02, Connector_JST:JST_XH_B02B-XH-A_1x02_P2.50mm_Vertical, B.Cu at (248.4, 66.3)
- added J8: Conn_01x02, Connector_JST:JST_XH_B02B-XH-A_1x02_P2.50mm_Vertical, B.Cu at (239.5, 66.3)
Connections:
- J3 pad 3: Net-(J3-Pad3) -> /Mode
- J4 pad 3: Net-(J4-Pad3) -> /RST
- J5 pad 3: Net-(J5-Pad3) -> /RST
- J5 pad 9: Net-(J5-Pad9) -> /Mode
Routing:
- net /RST: track 0.00 -> 100.3 mm
- net /Mode: track 0.00 -> 82.3 mm
- net /Col2: track 261.8 -> 317.1 mm
- net /Col1: track 287.9 -> 315.2 mm
- net /Col3: track 238.0 -> 258.4 mm
- net /Row1: track 283.0 -> 263.6 mm
- net /Row6: track 212.6 -> 199.1 mm
- net /Col5: track 167.1 -> 157.5 mm
- net /Col4: track 216.7 -> 209.2 mm
- net /Col6: track 142.6 -> 138.1 mm
- net /Row5: track 302.6 -> 306.5 mm
- net /Row2: track 259.0 -> 261.3 mm
- net /Row3: track 282.7 -> 280.5 mm
- net GND: track 0.00 -> 1.45 mm
Other:
- board text added: "Mode"
- board text added: "RST"

Commit message: Updating everything
Other:
- board size 257.7 x 65.9 mm -> 257.7 x 66.9 mm
