File: A-10CV1.2/A-10C-UFC/A-10C-UFC.kicad_pcb (KiCad board)
At the start: 2 copper layers, 257.7 x 66.9 mm, 45 parts, among them J1 Conn_01x08_MountingPin, J2 Conn_01x10_MountingPin, J3 Conn_01x06_MountingPin, J4 Conn_01x15_Female, J5 Conn_01x15_Female, J6 Conn_01x08_MountingPin, J7 Conn_01x02, J8 Conn_01x02, SW1 SW_Push, SW10 SW_Push, SW11 SW_Push, SW12 SW_Push, SW13 SW_Push, SW14 SW_Push, SW15 SW_Push, SW16 SW_Push, SW17 SW_Push, SW18 SW_Push, SW19 SW_Push, SW2 SW_Push, SW20 SW_Push, SW21 SW_Push, SW22 SW_Push, SW23 SW_Push, SW24 SW_Push, SW25 SW_Push, SW26 SW_Push, SW27 SW_Push, SW28 SW_Push, SW29 SW_Push, SW3 SW_Push, SW30 SW_Push, SW31 SW_Push, SW32 SW_Push, SW33 SW_Push, SW34 SW_Push, SW35 SW_Push, SW4 SW_Push, SW5 SW_Push, SW6 SW_Push, SW7 SW_Push, SW8 SW_Push, SW9 SW_Push

Commit message: more revisions
Other:
- board text added: "Nano Socket Pin 1 indicated by triangle (duh)"

Commit message: Always tweaking board shapes.
Parts:
- R1: moved to B.Cu
- moved R1 7.37 mm to (229.6, 67.7), turned to 270 degrees
- moved J1 4.89 mm to (256.8, 115.1)
- moved J2 4.89 mm to (278.6, 115.1)
- moved J3 4.89 mm to (256.8, 67.1)
- moved J4 4.89 mm to (211.1, 80.4)
- moved J5 4.89 mm to (211.1, 95.6)
- moved J7 4.89 mm to (243.6, 67.1)
- moved J8 4.89 mm to (234.7, 67.1)
- moved J6 4.89 mm to (274.6, 67.1)
Routing:
- net /Col2: track 317.1 -> 259.3 mm
- net /Row5: track 306.5 -> 350.7 mm
- net /Col3: track 258.4 -> 291.0 mm
- net /Col1: track 315.2 -> 286.6 mm, vias 0 -> 1
- net /Row6: track 199.1 -> 222.6 mm
- net /Mode: track 82.3 -> 59.0 mm, vias 0 -> 1
- net GND: track 1.45 -> 15.7 mm, vias 0 -> 2
- net /Col4: track 209.2 -> 222.7 mm
- net /Row3: track 280.5 -> 270.4 mm
- net /MastCaut: track 90.7 -> 98.1 mm
- net /RST: track 100.3 -> 93.5 mm
- net /Row4: track 315.7 -> 310.2 mm
- net /Row1: track 263.6 -> 268.6 mm
- net /Col5: track 157.5 -> 162.4 mm
- net /Col6: track 138.1 -> 141.3 mm
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Other:
- board size 257.7 x 66.9 mm -> 258.2 x 69.1 mm

Commit message: Updated PCB to move headers further inboard from edge
Parts:
- SW1, SW10, SW11, SW12, SW13, SW14, SW15, SW16, SW17, SW18, SW19, SW2, SW20, SW21, SW22, SW23, SW24, SW25, SW26, SW27, SW28, SW29, SW3, SW30, SW31, SW32, SW33, SW34, SW35, SW4, SW5, SW6, SW7, SW8, SW9: footprint Buttons_Switches_THT:SW_PUSH_6mm -> Button_Switch_THT:SW_PUSH_6mm
- moved J4 2.59 mm to (208.5, 80.4)
- moved J5 2.59 mm to (208.5, 95.6)
- moved J6 2.59 mm to (272.0, 67.1)
- moved J1 2.59 mm to (254.2, 115.1)
- moved J3 2.59 mm to (254.2, 67.1)
- moved J2 2.59 mm to (276.0, 115.1)
Routing:
- net GND: track 15.7 -> 93.2 mm, vias 2 -> 5
- net /Col3: track 291.0 -> 221.4 mm
- net /Row5: track 350.7 -> 298.5 mm
- net /MastCaut: track 98.1 -> 84.0 mm, vias 0 -> 1
- net /Row3: track 270.4 -> 283.2 mm
- net /Row2: track 262.0 -> 252.2 mm
- net /Row4: track 310.2 -> 319.9 mm, vias 0 -> 1
- net /Row6: track 222.6 -> 212.9 mm
- net /Col5: track 162.4 -> 171.3 mm
- net /RST: track 93.5 -> 101.8 mm
- net /Col2: track 259.3 -> 251.2 mm
- net /Mode: track 59.0 -> 57.2 mm, vias 1 -> 0
- net /Col1: track 286.6 -> 285.1 mm, vias 1 -> 0
- net /Col4: track 222.7 -> 224.1 mm
- net /Row1: track 268.6 -> 269.4 mm

Commit message: Always finding little imperfections.
Routing:
- net /Col3: track 221.4 -> 281.3 mm
- net /Row5: track 298.5 -> 325.8 mm
- net /Mode: track 57.2 -> 73.6 mm
- net /Row3: track 283.2 -> 267.0 mm, vias 0 -> 1
- net /Col5: track 171.3 -> 158.9 mm
- net /MastCaut: track 84.0 -> 95.4 mm, vias 1 -> 0
- net /Row1: track 269.4 -> 278.6 mm
- net GND: track 93.2 -> 84.8 mm, vias 5 -> 0
- net /Row4: track 319.9 -> 328.0 mm, vias 1 -> 0
- net /Col6: track 141.6 -> 146.2 mm
- net /Row6: track 212.9 -> 216.8 mm, vias 0 -> 1
- net Net-(D1-Pad1): track 9.92 -> 13.5 mm
- net /Row2: track 252.2 -> 255.5 mm, vias 1 -> 0
- net /Col2: track 251.2 -> 252.8 mm, vias 0 -> 1
- net /Col4: track 224.1 -> 222.5 mm
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