File: A-10CV1.2/A-10C-UFC/A-10C-UFC.sch (KiCad schematic (older format))
At the start: 47 parts, among them J1 Conn_01x08_MountingPin, J2 Conn_01x10_MountingPin, J3 Conn_01x06_MountingPin, J4 Conn_01x15_Female, J5 Conn_01x15_Female, J6 Conn_01x08_MountingPin, J7 Conn_01x02, J8 Conn_01x02, SW1 SW_Push, SW10 SW_Push, SW11 SW_Push, SW12 SW_Push, SW13 SW_Push, SW14 SW_Push, SW15 SW_Push, SW16 SW_Push, SW17 SW_Push, SW18 SW_Push, SW19 SW_Push, SW2 SW_Push, SW20 SW_Push, SW21 SW_Push, SW22 SW_Push, SW23 SW_Push, SW24 SW_Push, SW25 SW_Push, SW26 SW_Push, SW27 SW_Push, SW28 SW_Push, SW29 SW_Push, SW3 SW_Push, SW30 SW_Push, SW31 SW_Push, SW32 SW_Push, SW33 SW_Push, SW34 SW_Push, SW35 SW_Push, SW36 SW_Push, SW37 SW_SPST, SW4 SW_Push, SW5 SW_Push, SW6 SW_Push, SW7 SW_Push, SW8 SW_Push, SW9 SW_Push

Commit message: Forgot some
Parts:
- J1, J6: symbol Connector_Generic_MountingPin:Conn_01x08_MountingPin -> A-10C-UFC-rescue:Conn_01x08_MountingPin-Connector_Generic_MountingPin
- J2: symbol Connector_Generic_MountingPin:Conn_01x10_MountingPin -> A-10C-UFC-rescue:Conn_01x10_MountingPin-Connector_Generic_MountingPin
- J3: symbol Connector_Generic_MountingPin:Conn_01x06_MountingPin -> A-10C-UFC-rescue:Conn_01x06_MountingPin-Connector_Generic_MountingPin
- J4, J5: symbol Connector:Conn_01x15_Female -> A-10C-UFC-rescue:Conn_01x15_Female-Connector
- J7, J8: symbol Connector_Generic:Conn_01x02 -> A-10C-UFC-rescue:Conn_01x02-Connector_Generic
- SW1, SW10, SW11, SW12, SW13, SW14, SW15, SW16, SW17, SW18, SW19, SW2, SW20, SW21, SW22, SW23, SW24, SW25, SW26, SW27, SW28, SW29, SW3, SW30, SW31, SW32, SW33, SW34, SW35, SW36, SW4, SW5, SW6, SW7, SW8, SW9: symbol Switch:SW_Push -> A-10C-UFC-rescue:SW_Push-Switch
- SW37: symbol Switch:SW_SPST -> A-10C-UFC-rescue:SW_SPST-Switch
Changed lines of the file:
@@
 $EndDescr
 $Comp
-L Switch:SW_Push SW1
+L A-10C-UFC-rescue:SW_Push-Switch SW1
 U 1 1 5D362DF4
 P 1950 1650
@@
 $EndComp
 $Comp
-L Switch:SW_Push SW7
+L A-10C-UFC-rescue:SW_Push-Switch SW7
 U 1 1 5D36336E
 P 2650 1650
@@
 $EndComp
 $Comp
-L Switch:SW_Push SW13
+L A-10C-UFC-rescue:SW_Push-Switch SW13
 U 1 1 5D3639C9
 P 3350 1650
@@
 $EndComp
 $Comp
-L Switch:SW_Push SW19
+L A-10C-UFC-rescue:SW_Push-Switch SW19
 U 1 1 5D363AC3
 P 4050 1650
@@
 $EndComp
 $Comp
-L Switch:SW_Push SW25
+L A-10C-UFC-rescue:SW_Push-Switch SW25
 U 1 1 5D363C5F
 P 4750 1650
@@
 $EndComp
 $Comp
-L Switch:SW_Push SW31
+L A-10C-UFC-rescue:SW_Push-Switch SW31
 U 1 1 5D363EE9
 P 5450 1650
@@
 $EndComp
 $Comp
-L Switch:SW_Push SW2
+L A-10C-UFC-rescue:SW_Push-Switch SW2
 U 1 1 5D36DD6D
 P 1950 2250
@@
 $EndComp
 $Comp
-L Switch:SW_Push SW8
+L A-10C-UFC-rescue:SW_Push-Switch SW8
 U 1 1 5D36DD73
 P 2650 2250
@@
 $EndComp
 $Comp
-L Switch:SW_Push SW14
+L A-10C-UFC-rescue:SW_Push-Switch SW14
 U 1 1 5D36DD79
 P 3350 2250
@@
 $EndComp
 $Comp
-L Switch:SW_Push SW20
+L A-10C-UFC-rescue:SW_Push-Switch SW20
 U 1 1 5D36DD7F
 P 4050 2250
@@
 $EndComp
 $Comp
-L Switch:SW_Push SW26
+L A-10C-UFC-rescue:SW_Push-Switch SW26
 U 1 1 5D36DD85
 P 4750 2250
@@
 $EndComp
 $Comp
-L Switch:SW_Push SW32
+L A-10C-UFC-rescue:SW_Push-Switch SW32
 U 1 1 5D36DD8B
 P 5450 2250
@@
 $EndComp
 $Comp
-L Switch:SW_Push SW3
+L A-10C-UFC-rescue:SW_Push-Switch SW3
 U 1 1 5D36F3B5
 P 1950 2900
@@
 $EndComp
 $Comp
-L Switch:SW_Push SW9
+L A-10C-UFC-rescue:SW_Push-Switch SW9
 U 1 1 5D36F3BB
 P 2650 2900
@@
 $EndComp
 $Comp
-L Switch:SW_Push SW15
+L A-10C-UFC-rescue:SW_Push-Switch SW15
 U 1 1 5D36F3C1
 P 3350 2900
@@
 $EndComp
 $Comp
-L Switch:SW_Push SW21
+L A-10C-UFC-rescue:SW_Push-Switch SW21
 U 1 1 5D36F3C7
 P 4050 2900
@@
 $EndComp
 $Comp
-L Switch:SW_Push SW27
+L A-10C-UFC-rescue:SW_Push-Switch SW27
 U 1 1 5D36F3CD
 P 4750 2900
@@
 $EndComp
 $Comp
-L Switch:SW_Push SW33
+L A-10C-UFC-rescue:SW_Push-Switch SW33
 U 1 1 5D36F3D3
 P 5450 2900
@@
 $EndComp
 $Comp
-L Switch:SW_Push SW4
+L A-10C-UFC-rescue:SW_Push-Switch SW4
 U 1 1 5D371E17
 P 1950 3500
@@
 $EndComp
 $Comp
-L Switch:SW_Push SW10
+L A-10C-UFC-rescue:SW_Push-Switch SW10
 U 1 1 5D371E1D
 P 2650 3500
@@
 $EndComp
 $Comp
-L Switch:SW_Push SW16
+L A-10C-UFC-rescue:SW_Push-Switch SW16
 U 1 1 5D371E23
 P 3350 3500
@@
 $EndComp
 $Comp
-L Switch:SW_Push SW22
+L A-10C-UFC-rescue:SW_Push-Switch SW22
 U 1 1 5D371E29
 P 4050 3500
@@
 $EndComp
 $Comp
-L Switch:SW_Push SW28
+L A-10C-UFC-rescue:SW_Push-Switch SW28
 U 1 1 5D371E2F
 P 4750 3500
@@
 $EndComp
 $Comp
-L Switch:SW_Push SW34
+L A-10C-UFC-rescue:SW_Push-Switch SW34
 U 1 1 5D371E35
 P 5450 3500
@@
 $EndComp
 $Comp
-L Switch:SW_Push SW5
+L A-10C-UFC-rescue:SW_Push-Switch SW5
 U 1 1 5D374755
 P 1950 4100
@@
 $EndComp
 $Comp
-L Switch:SW_Push SW11
+L A-10C-UFC-rescue:SW_Push-Switch SW11
 U 1 1 5D37475B
 P 2650 4100
@@
 $EndComp
 $Comp
-L Switch:SW_Push SW17
+L A-10C-UFC-rescue:SW_Push-Switch SW17
 U 1 1 5D374761
 P 3350 4100
@@
 $EndComp
 $Comp
-L Switch:SW_Push SW23
+L A-10C-UFC-rescue:SW_Push-Switch SW23
 U 1 1 5D374767
 P 4050 4100
@@
 $EndComp
 $Comp
-L Switch:SW_Push SW29
+L A-10C-UFC-rescue:SW_Push-Switch SW29
 U 1 1 5D37476D
 P 4750 4100
@@
 $EndComp
 $Comp
-L Switch:SW_Push SW35
+L A-10C-UFC-rescue:SW_Push-Switch SW35
 U 1 1 5D374773
 P 5450 4100
@@
 Row5
 $Comp
-L Switch:SW_Push SW6
+L A-10C-UFC-rescue:SW_Push-Switch SW6
 U 1 1 5D3990F4
 P 1950 4800
@@
 $EndComp
 $Comp
-L Switch:SW_Push SW12
+L A-10C-UFC-rescue:SW_Push-Switch SW12
 U 1 1 5D3990FA
 P 2650 4800
@@
 $EndComp
 $Comp
-L Switch:SW_Push SW18
+L A-10C-UFC-rescue:SW_Push-Switch SW18
 U 1 1 5D399100
 P 3350 4800
@@
 $EndComp
 $Comp
-L Switch:SW_Push SW24
+L A-10C-UFC-rescue:SW_Push-Switch SW24
 U 1 1 5D399106
 P 4050 4800
@@
 $EndComp
 $Comp
-L Switch:SW_Push SW30
+L A-10C-UFC-rescue:SW_Push-Switch SW30
 U 1 1 5D39910C
 P 4750 4800
@@
 	5650 4100 5650 5500
 $Comp
-L Connector_Generic_MountingPin:Conn_01x08_MountingPin J1
+L A-10C-UFC-rescue:Conn_01x08_MountingPin-Connector_Generic_MountingPin J1
 U 1 1 5D3E5163
 P 7600 3800
@@
 $EndComp
 $Comp
-L Connector_Generic_MountingPin:Conn_01x10_MountingPin J2
+L A-10C-UFC-rescue:Conn_01x10_MountingPin-Connector_Generic_MountingPin J2
 U 1 1 5D3E89EE
 P 7600 5000
@@
 $EndComp
 $Comp
-L Connector_Generic_MountingPin:Conn_01x06_MountingPin J3
+L A-10C-UFC-rescue:Conn_01x06_MountingPin-Connector_Generic_MountingPin J3
 U 1 1 5D3E9A00
 P 8900 3700
@@
 $EndComp
 $Comp
-L power:GND #PWR01
+L A-10C-UFC-rescue:GND-power #PWR01
 U 1 1 5D434D02
 P 7800 1650
@@
 A0
 $Comp
-L Connector:Conn_01x15_Female J4
+L A-10C-UFC-rescue:Conn_01x15_Female-Connector J4
 U 1 1 5D42500E
 P 11250 1650
@@
 $EndComp
 $Comp
-L Connector:Conn_01x15_Female J5
+L A-10C-UFC-rescue:Conn_01x15_Female-Connector J5
 U 1 1 5D4252F1
 P 11250 3350
@@
 NoConn ~ 7000 5100
 $Comp
-L Connector_Generic:Conn_01x02 J7
+L A-10C-UFC-rescue:Conn_01x02-Connector_Generic J7
 U 1 1 5D473A0F
 P 11300 4750
@@
 $EndComp
 $Comp
-L Connector_Generic:Conn_01x02 J8
+L A-10C-UFC-rescue:Conn_01x02-Connector_Generic J8
 U 1 1 5D473B23
 P 11300 5350
@@
 $EndComp
 $Comp
-L Switch:SW_Push SW36
+L A-10C-UFC-rescue:SW_Push-Switch SW36
 U 1 1 5D473BB8
 P 10700 4750
@@
 $EndComp
 $Comp
-L Switch:SW_SPST SW37
+L A-10C-UFC-rescue:SW_SPST-Switch SW37
 U 1 1 5D473C67
 P 10700 5350
@@
 GND
 $Comp
-L Connector_Generic_MountingPin:Conn_01x08_MountingPin J6
+L A-10C-UFC-rescue:Conn_01x08_MountingPin-Connector_Generic_MountingPin J6
 U 1 1 5D4991C7
 P 8900 4900

Commit message: Added new designs for a Caution Lights Panel.
Parts:
- R1: value R -> 220
Changed lines of the file:
@@
 P 7400 1450
 F 0 "R1" V 7193 1450 50  0000 C CNN
-F 1 "R" V 7284 1450 50  0000 C CNN
+F 1 "220" V 7284 1450 50  0000 C CNN
 F 2 "Resistor_THT:R_Axial_DIN0207_L6.3mm_D2.5mm_P7.62mm_Horizontal" V 7330 1450 50  0001 C CNN
 F 3 "~" H 7400 1450 50  0001 C CNN
